Commit message: Fix base_link Z height

File: my_robot/urdf/my_robot.xacro (robot description, xacro)
@@ -4,5 +4,5 @@
   <link name="base_link"></link>
   <joint name="base_link_joint" type="fixed">
-    <origin xyz="0 0 0" rpy="0 0 0"/>
+    <origin xyz="0 0 0.11" rpy="0 0 0"/>
     <parent link="base_link"/>
     <child link="chassis"/>
